File: system_development/Prototyping_24/PCB files/Pump Power PCB/Pump Power PCB.kicad_pcb (KiCad board)
At the start: 2 copper layers, 34.9 x 24.8 mm, 3 parts, among them J1 Barrel_Jack, J2 Positive Terminal, J3 Negative Terminal

Commit message: Altered PCB's
Parts:
- added REF**: 2.2 mm Drill Hole, Custom Footprints:2.2 mm Drill Hole, F.Cu at (158.1, 108.6)
- added REF**: 2.2 mm Drill Hole, Custom Footprints:2.2 mm Drill Hole, F.Cu at (133.3, 78.7)
Other:
- board size 34.9 x 24.8 mm -> 34.9 x 34.9 mm
- board text added: "M2"
Changed lines of the file:
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@@
     )
+  )
+  (footprint "Custom Footprints:2.2 mm Drill Hole" (layer "F.Cu")
+    (at 158.115 108.585)
+    (attr through_hole)
+    (fp_text reference "REF**" (at 0 -0.5 unlocked) (layer "F.SilkS") hide
+        (effects (font (size 1 1) (thickness 0.1)))
+    )
+    (fp_text value "2.2 mm Drill Hole" (at 0 1 unlocked) (layer "F.Fab")
+        (effects (font (size 1 1) (thickness 0.15)))
+    )
+    (fp_text user "${REFERENCE}" (at 0 2.5 unlocked) (layer "F.Fab")
+        (effects (font (size 1 1) (thickness 0.15)))
+    )
+    (pad "" np_thru_hole circle (at 0 0) (size 2.5 2.5) (drill 2.2) (layers "F&B.Cu" "*.Mask"))
   )
   (footprint "TerminalBlock_Phoenix:TerminalBlock_Phoenix_MKDS-1,5-2-5.08_1x02_P5.08mm_Horizontal" (layer "F.Cu")
@@
     )
   )
+  (footprint "Custom Footprints:2.2 mm Drill Hole" (layer "F.Cu")
+    (at 133.35 78.74)
+    (attr through_hole)
+    (fp_text reference "REF**" (at 0 -0.5 unlocked) (layer "F.SilkS") hide
+        (effects (font (size 1 1) (thickness 0.1)))
+    )
+    (fp_text value "2.2 mm Drill Hole" (at 0 1 unlocked) (layer "F.Fab")
+        (effects (font (size 1 1) (thickness 0.15)))
+    )
+    (fp_text user "${REFERENCE}" (at 0 2.5 unlocked) (layer "F.Fab")
+        (effects (font (size 1 1) (thickness 0.15)))
+    )
+    (pad "" np_thru_hole circle (at 0 0) (size 2.5 2.5) (drill 2.2) (layers "F&B.Cu" "*.Mask"))
+  )
+  (gr_line (start 142.24 80.645) (end 144.145 81.28)
+    (stroke (width 0.1) (type default)) (layer "Edge.Cuts"))
+  (gr_line (start 128.27 81.28) (end 128.27 76.2)
+    (stroke (width 0.1) (type default)) (layer "Edge.Cuts"))
+  (gr_line (start 128.27 106.045) (end 149.86 106.045)
+    (stroke (width 0.1) (type default)) (layer "Edge.Cuts"))
+  (gr_line (start 163.195 111.125) (end 154.305 111.125)
+    (stroke (width 0.1) (type default)) (layer "Edge.Cuts"))
+  (gr_line (start 128.27 76.2) (end 137.16 76.2)
+    (stroke (width 0.1) (type default)) (layer "Edge.Cuts"))
+  (gr_line (start 137.16 76.2) (end 142.24 80.645)
+    (stroke (width 0.1) (type default)) (layer "Edge.Cuts"))
+  (gr_line (start 154.305 111.125) (end 149.86 106.045)
+    (stroke (width 0.1) (type default)) (layer "Edge.Cuts"))
   (gr_line (start 163.195 81.28) (end 163.195 106.045)
     (stroke (width 0.1) (type default)) (layer "Edge.Cuts"))
-  (gr_line (start 163.195 106.045) (end 128.27 106.045)
+  (gr_line (start 163.195 106.045) (end 163.195 111.125)
     (stroke (width 0.1) (type default)) (layer "Edge.Cuts"))
-  (gr_line (start 128.27 81.28) (end 163.195 81.28)
+  (gr_line (start 144.145 81.28) (end 163.195 81.28)
     (stroke (width 0.1) (type default)) (layer "Edge.Cuts"))
   (gr_line (start 128.27 106.045) (end 128.27 81.28)
@@
     (effects (font (size 1 1) (thickness 0.15)) (justify left bottom mirror))
   )
+  (gr_text "M2" (at 129.54 79.375) (layer "F.SilkS")
+    (effects (font (size 1 1) (thickness 0.15)) (justify left bottom))
+  )
+  (gr_text "M2" (at 154.305 109.22) (layer "F.SilkS")
+    (effects (font (size 1 1) (thickness 0.15)) (justify left bottom))
+  )
   (segment (start 143.77 96.145) (end 137.795 90.17) (width 0.25) (layer "F.Cu") (net 1))
